File: steno-keyboard.kicad_pcb (KiCad board)
At the start: 2 copper layers, 0 parts

Commit message: Updated PCB and footprints
Parts:
- added A1: RaspberryPi_Pico, Module:RaspberryPi_Pico_Common_Unspecified, F.Cu at (47.0, 134.6)
- added SW1: SW_Push, MX_Solderable:MX-Solderable-1U, F.Cu at (133.3, 38.1)
- added SW10: SW_Push, MX_Solderable:MX-Solderable-1U, F.Cu at (342.9, 38.1)
- added SW11: SW_Push, MX_Solderable:MX-Solderable-1U, F.Cu at (361.9, 38.1)
- added SW12: SW_Push, MX_Solderable:MX-Solderable-1U, F.Cu at (152.4, 57.1)
- added SW13: SW_Push, MX_Solderable:MX-Solderable-1U, F.Cu at (171.4, 57.1)
- added SW14: SW_Push, MX_Solderable:MX-Solderable-1U, F.Cu at (190.5, 57.1)
- added SW15: SW_Push, MX_Solderable:MX-Solderable-1U, F.Cu at (285.8, 57.1)
- added SW16: SW_Push, MX_Solderable:MX-Solderable-1U, F.Cu at (304.8, 57.1)
- added SW17: SW_Push, MX_Solderable:MX-Solderable-1U, F.Cu at (323.9, 57.1)
- added SW18: SW_Push, MX_Solderable:MX-Solderable-1U, F.Cu at (342.9, 57.1)
- added SW19: SW_Push, MX_Solderable:MX-Solderable-1U, F.Cu at (361.9, 57.1)
- added SW2: SW_Push, MX_Solderable:MX-Solderable-1U, F.Cu at (152.4, 38.1)
- added SW20: SW_Push, MX_Solderable:MX-Solderable-1U, F.Cu at (171.4, 95.2)
- added SW21: SW_Push, MX_Solderable:MX-Solderable-1U, F.Cu at (190.5, 95.2)
- added SW22: SW_Push, MX_Solderable:MX-Solderable-1U, F.Cu at (209.6, 95.2)
- added SW23: SW_Push, MX_Solderable:MX-Solderable-1U, F.Cu at (266.7, 95.2)
- added SW24: SW_Push, MX_Solderable:MX-Solderable-1U, F.Cu at (285.8, 95.2)
- added SW25: SW_Push, MX_Solderable:MX-Solderable-1U, F.Cu at (304.8, 95.2)
- added SW3: SW_Push, MX_Solderable:MX-Solderable-1U, F.Cu at (171.4, 38.1)
- added SW4: SW_Push, MX_Solderable:MX-Solderable-1U, F.Cu at (190.5, 38.1)
- added SW5: SW_Push, MX_Solderable:MX-Solderable-1U, F.Cu at (209.6, 38.1)
- added SW6: SW_Push, MX_Solderable:MX-Solderable-1U, F.Cu at (266.7, 38.1)
- added SW7: SW_Push, MX_Solderable:MX-Solderable-1U, F.Cu at (285.8, 38.1)
- added SW8: SW_Push, MX_Solderable:MX-Solderable-1U, F.Cu at (304.8, 38.1)
- added SW9: SW_Push, MX_Solderable:MX-Solderable-1U, F.Cu at (323.9, 38.1)
